File: pcb/hardware/fourth.kicad_sch (KiCad schematic)
At the start: 83 parts, among them J1 Conn_01x04, J10 Conn_01x04, J11 Conn_01x04, J12 Conn_01x06, J3 USB_B_Micro, J5 Conn_01x04, J6 Conn_01x06, J7 Conn_01x03_Pin, J8 Conn_01x03_Pin, J9 Conn_01x04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

Commit message: Update pcb
Parts:
- J1, J10, J11, J5, J9: footprint Connector_PinSocket_2.00mm:PinSocket_1x04_P2.00mm_Vertical -> Connector_JST:JST_ZH_B4B-ZR_1x04_P1.50mm_Vertical
- J12, J6: footprint Connector_PinSocket_2.00mm:PinSocket_1x06_P2.00mm_Vertical -> Connector_JST:JST_ZH_B6B-ZR_1x06_P1.50mm_Vertical
- J7, J8: footprint Connector_PinSocket_2.00mm:PinSocket_1x03_P2.00mm_Vertical -> Connector_JST:JST_ZH_B3B-ZR_1x03_P1.50mm_Vertical
Connections:
- net BUCK_IN is gone; now on net V: C24.1, C26.1, FB2.2, U6.2 (EN), U6.3 (IN)
Changed lines of the file:
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@@
 	)
 	(junction
+		(at 212.09 26.67)
+		(diameter 0)
+		(color 0 0 0 0)
+	)
+	(junction
 		(at 21.59 17.78)
 		(diameter 0)
@@
 	(wire
 		(pts
-			(xy 209.55 26.67) (xy 215.9 26.67)
+			(xy 209.55 26.67) (xy 212.09 26.67)
 		)
 		(stroke
@@
 	(wire
 		(pts
+			(xy 212.09 26.67) (xy 215.9 26.67)
+		)
+		(stroke
+			(width 0)
+			(type default)
+		)
+	)
+	(wire
+		(pts
 			(xy 237.49 31.75) (xy 259.08 31.75)
 		)
@@
 	(wire
 		(pts
+			(xy 212.09 19.05) (xy 212.09 26.67)
+		)
+		(stroke
+			(width 0)
+			(type default)
+		)
+	)
+	(wire
+		(pts
 			(xy 21.59 19.05) (xy 21.59 17.78)
 		)
@@
 		)
 	)
+	(global_label "V"
+		(shape input)
+		(at 212.09 19.05 90)
+		(fields_autoplaced yes)
+		(effects
+			(font
+				(size 1.27 1.27)
+			)
+			(justify left)
+		)
+		(property "Intersheetrefs" "${INTERSHEET_REFS}"
+			(at 212.09 14.9762 90)
+			(effects
+				(font
+					(size 1.27 1.27)
+				)
+				(justify left)
+				(hide yes)
+			)
+		)
+	)
 	(global_label "VIDEO_OUT"
 		(shape input)
@@
 			)
 		)
-		(property "Footprint" "Connector_PinSocket_2.00mm:PinSocket_1x04_P2.00mm_Vertical"
+		(property "Footprint" "Connector_JST:JST_ZH_B4B-ZR_1x04_P1.50mm_Vertical"
 			(at 55.88 156.21 0)
 			(effects
@@
 			)
 		)
-		(property "Footprint" "Connector_PinSocket_2.00mm:PinSocket_1x06_P2.00mm_Vertical"
+		(property "Footprint" "Connector_JST:JST_ZH_B6B-ZR_1x06_P1.50mm_Vertical"
 			(at 54.61 179.07 0)
 			(effects
@@
 			)
 		)
-		(property "Footprint" "Connector_PinSocket_2.00mm:PinSocket_1x04_P2.00mm_Vertical"
+		(property "Footprint" "Connector_JST:JST_ZH_B4B-ZR_1x04_P1.50mm_Vertical"
 			(at 78.74 156.21 0)
 			(effects
@@
 			)
 		)
-		(property "Footprint" "Connector_PinSocket_2.00mm:PinSocket_1x06_P2.00mm_Vertical"
+		(property "Footprint" "Connector_JST:JST_ZH_B6B-ZR_1x06_P1.50mm_Vertical"
 			(at 130.81 154.94 0)
 			(effects
@@
 			)
 		)
-		(property "Footprint" "Connector_PinSocket_2.00mm:PinSocket_1x04_P2.00mm_Vertical"
+		(property "Footprint" "Connector_JST:JST_ZH_B4B-ZR_1x04_P1.50mm_Vertical"
 			(at 26.67 156.21 0)
 			(effects
@@
 			)
 		)
-		(property "Footprint" "Connector_PinSocket_2.00mm:PinSocket_1x03_P2.00mm_Vertical"
+		(property "Footprint" "Connector_JST:JST_ZH_B3B-ZR_1x03_P1.50mm_Vertical"
 			(at 106.68 182.88 0)
 			(effects
@@
 			)
 		)
-		(property "Footprint" "Connector_PinSocket_2.00mm:PinSocket_1x03_P2.00mm_Vertical"
+		(property "Footprint" "Connector_JST:JST_ZH_B3B-ZR_1x03_P1.50mm_Vertical"
 			(at 107.95 156.21 0)
 			(effects
@@
 			)
 		)
-		(property "Footprint" "Connector_PinSocket_2.00mm:PinSocket_1x04_P2.00mm_Vertical"
+		(property "Footprint" "Connector_JST:JST_ZH_B4B-ZR_1x04_P1.50mm_Vertical"
 			(at 33.02 134.62 0)
 			(effects
@@
 			)
 		)
-		(property "Footprint" "Connector_PinSocket_2.00mm:PinSocket_1x04_P2.00mm_Vertical"
+		(property "Footprint" "Connector_JST:JST_ZH_B4B-ZR_1x04_P1.50mm_Vertical"
 			(at 78.74 180.34 0)
 			(effects
